File: gpio-expander.kicad_sch (KiCad schematic)
At the start: 5 parts, among them U1 TPS4H160AQPWPRQ1, U2 TPS4H160AQPWPRQ1, U3 TPS4H160AQPWPRQ1, U4 TPS4H160AQPWPRQ1, U5 MCP23017T-E_SO

Commit message: first pcb revision
Parts:
- added C1: C, Capacitor_SMD:C_0805_2012Metric_Pad1.18x1.45mm_HandSolder, symbol Device:C
- added D1, D10, D11, D12, D13, D14, D15, D16, D2, D3, D4, D5, D6, D7, D8, D9: 60V 1A, Diode_SMD:D_SOD-323_HandSoldering, symbol Device:D
- added H1, H2, H3, H4: MountingHole_Pad, MountingHole:MountingHole_3.2mm_M3_Pad_Via, symbol Mechanical:MountingHole_Pad
- added J1: Conn_01x04, Connector_PinHeader_2.54mm:PinHeader_1x04_P2.54mm_Vertical, symbol Connector_Generic:Conn_01x04
- added J2, J3, J4, J5: Conn_01x06, Connector_Samtec_HPM_THT:Samtec_HPM-06-05-x-S_Straight_1x06_Pitch5.08mm, symbol Connector_Generic:Conn_01x06
- added J6: Conn_01x04, Connector_Samtec_HPM_THT:Samtec_HPM-04-05-x-S_Straight_1x04_Pitch5.08mm, symbol Connector_Generic:Conn_01x04
- added JP1, JP2, JP3: SolderJumper_3_Open, Jumper:SolderJumper-3_P1.3mm_Open_RoundedPad1.0x1.5mm, symbol Jumper:SolderJumper_3_Open
- added R1, R2, R3, R4: R, Resistor_SMD:R_0603_1608Metric_Pad0.98x0.95mm_HandSolder, symbol Device:R
Connections:
- net GND: now reaches U3.1 (GND), U3.12 (GND)
- net GND: now also U1.1 (GND), U1.12 (GND), U1.29 (EXP), U1.30 (EXP), U1.31 (EXP), U1.32 (EXP), U1.33 (EXP), U1.34 (EXP), U1.35 (EXP), U1.36 (EXP), U1.37 (EXP), U1.38 (EXP), U1.39 (EXP), U1.40 (EXP), U1.41 (EXP), U1.42 (EXP), U1.43 (EXP), U1.44 (EXP), U1.45 (EXP), U1.46 (EXP), U1.47 (EXP), U1.48 (EXP), U1.49 (EXP), U1.50 (EXP), U1.51 (EXP), U1.52 (EXP), U1.53 (EXP), U2.1 (GND), U2.12 (GND), U2.29 (EXP), U2.30 (EXP), U2.31 (EXP), U2.32 (EXP), U2.33 (EXP), U2.34 (EXP), U2.35 (EXP), U2.36 (EXP), U2.37 (EXP), U2.38 (EXP), U2.39 (EXP), U2.40 (EXP), U2.41 (EXP), U2.42 (EXP), U2.43 (EXP), U2.44 (EXP), U2.45 (EXP), U2.46 (EXP), U2.47 (EXP), U2.48 (EXP), U2.49 (EXP), U2.50 (EXP), U2.51 (EXP), U2.52 (EXP), U2.53 (EXP), U3.29 (EXP), U3.30 (EXP), U3.31 (EXP), U3.32 (EXP), U3.33 (EXP), U3.34 (EXP), U3.35 (EXP), U3.36 (EXP), U3.37 (EXP), U3.38 (EXP), U3.39 (EXP), U3.40 (EXP), U3.41 (EXP), U3.42 (EXP), U3.43 (EXP), U3.44 (EXP), U3.45 (EXP), U3.46 (EXP), U3.47 (EXP), U3.48 (EXP), U3.49 (EXP), U3.50 (EXP), U3.51 (EXP), U3.52 (EXP), U3.53 (EXP), U4.1 (GND), U4.12 (GND), U4.29 (EXP), U4.30 (EXP), U4.31 (EXP), U4.32 (EXP), U4.33 (EXP), U4.34 (EXP), U4.35 (EXP), U4.36 (EXP), U4.37 (EXP), U4.38 (EXP), U4.39 (EXP), U4.40 (EXP), U4.41 (EXP), U4.42 (EXP), U4.43 (EXP), U4.44 (EXP), U4.45 (EXP), U4.46 (EXP), U4.47 (EXP), U4.48 (EXP), U4.49 (EXP), U4.50 (EXP), U4.51 (EXP), U4.52 (EXP), U4.53 (EXP), U5.10 (VSS), C1.2, D1.2 (A), D10.2 (A), D11.2 (A), D12.2 (A), D13.2 (A), D14.2 (A), D15.2 (A), D16.2 (A), D2.2 (A), D3.2 (A), D4.2 (A), D5.2 (A), D6.2 (A), D7.2 (A), D8.2 (A), D9.2 (A), H1.1, H2.1, H3.1, H4.1, J1.1 (Pin_1), J2.1 (Pin_1), J2.6 (Pin_6), J3.1 (Pin_1), J3.6 (Pin_6), J4.1 (Pin_1), J4.6 (Pin_6), J5.1 (Pin_1), J5.6 (Pin_6), J6.3 (Pin_3), J6.4 (Pin_4), JP1.3 (B), JP2.3 (B), JP3.3 (B), R1.1, R2.1, R3.1, R4.1
- net at U3.11 (CL): now also R2.2
- net at U3.15 (OUT4), U3.16 (OUT4): now also D4.1 (K), J3.5 (Pin_5)
- net at U3.17 (OUT3), U3.18 (OUT3): now also D3.1 (K), J3.4 (Pin_4)
- net +24V: now reaches U3.20 (VS), U3.21 (VS), U3.22 (VS), U3.23 (VS)
- net +24V: now also U1.20 (VS), U1.21 (VS), U1.22 (VS), U1.23 (VS), U2.20 (VS), U2.21 (VS), U2.22 (VS), U2.23 (VS), U4.20 (VS), U4.21 (VS), U4.22 (VS), U4.23 (VS), J6.1 (Pin_1), J6.2 (Pin_2)
- net at U3.25 (OUT2), U3.26 (OUT2): now also D2.1 (K), J3.3 (Pin_3)
- net at U3.27 (OUT1), U3.28 (OUT1): now also D1.1 (K), J3.2 (Pin_2)
- net at U3.3 (IN1): now also U5.28 (GPA7); no longer U5.1 (GPB0)
- net at U3.4 (IN2): now also U5.27 (GPA6); no longer U5.2 (GPB1)
- net at U3.5 (IN3): now also U5.26 (GPA5); no longer U5.3 (GPB2)
- net at U3.6 (IN4): now also U5.25 (GPA4); no longer U5.4 (GPB3)
- net at U1.11 (CL): now also R4.2
- net at U1.15 (OUT4), U1.16 (OUT4): now also D12.1 (K), J4.5 (Pin_5)
- net at U1.17 (OUT3), U1.18 (OUT3): now also D11.1 (K), J4.4 (Pin_4)
- net at U1.25 (OUT2), U1.26 (OUT2): now also D10.1 (K), J4.3 (Pin_3)
- net at U1.27 (OUT1), U1.28 (OUT1): now also D9.1 (K), J4.2 (Pin_2)
- net at U1.3 (IN1): now also U5.8 (GPB7); no longer U5.21 (GPA0)
- net at U1.4 (IN2): now also U5.7 (GPB6); no longer U5.22 (GPA1)
- net at U1.5 (IN3): now also U5.6 (GPB5); no longer U5.23 (GPA2)
- net at U1.6 (IN4): now also U5.5 (GPB4); no longer U5.24 (GPA3)
- net at U4.11 (CL): now also R1.2
- net at U4.15 (OUT4), U4.16 (OUT4): now also D5.1 (K), J2.5 (Pin_5)
- net at U4.17 (OUT3), U4.18 (OUT3): now also D6.1 (K), J2.4 (Pin_4)
- net at U4.25 (OUT2), U4.26 (OUT2): now also D7.1 (K), J2.3 (Pin_3)
- net at U4.27 (OUT1), U4.28 (OUT1): now also D8.1 (K), J2.2 (Pin_2)
- net at U4.3 (IN1): now also U5.24 (GPA3); no longer U5.5 (GPB4)
- net at U4.4 (IN2): now also U5.23 (GPA2); no longer U5.6 (GPB5)
- net at U4.5 (IN3): now also U5.22 (GPA1); no longer U5.7 (GPB6)
- net at U4.6 (IN4): now also U5.21 (GPA0); no longer U5.8 (GPB7)
- net at U2.11 (CL): now also R3.2
- net at U2.15 (OUT4), U2.16 (OUT4): now also D16.1 (K), J5.5 (Pin_5)
- net at U2.17 (OUT3), U2.18 (OUT3): now also D15.1 (K), J5.4 (Pin_4)
- net at U2.25 (OUT2), U2.26 (OUT2): now also D14.1 (K), J5.3 (Pin_3)
- net at U2.27 (OUT1), U2.28 (OUT1): now also D13.1 (K), J5.2 (Pin_2)
- net at U2.3 (IN1): now also U5.4 (GPB3); no longer U5.25 (GPA4)
- net at U2.4 (IN2): now also U5.3 (GPB2); no longer U5.26 (GPA5)
- net at U2.5 (IN3): now also U5.2 (GPB1); no longer U5.27 (GPA6)
- net at U2.6 (IN4): now also U5.1 (GPB0); no longer U5.28 (GPA7)
- net at U5.12 (SCK): now also J1.2 (Pin_2)
- net at U5.13 (SDA): now also J1.3 (Pin_3)
- net at U5.15 (A0): now also JP1.2 (C)
- net at U5.16 (A1): now also JP2.2 (C)
- net at U5.17 (A2): now also JP3.2 (C)
- net +3V3: now reaches U5.18 (~{RESET})
- net +3V3: now also U5.9 (VDD), C1.1, J1.4 (Pin_4), JP1.1 (A), JP2.1 (A), JP3.1 (A)
- no-connect marks 0 -> 26
Other:
- moved on the sheet: U1, U2, U3, U4
